Commit message: Adjusted wheel track and lidar height

File: rover_ws/src/rover_bringup/urdf/rover.urdf (robot description, URDF)
Before this commit: robot rover, 3 links, 2 joints
Links:
- added link left_wheel
- added link right_wheel
Joints:
- added joint base_to_left_wheel: type continuous, parent base_link, child left_wheel, origin xyz=0 0.09 0 rpy=-1.5708 0 0, axis 0 0 1
- added joint base_to_right_wheel: type continuous, parent base_link, child right_wheel, origin xyz=0 -0.09 0 rpy=-1.5708 0 0, axis 0 0 1
- joint base_to_laser: origin xyz=0 0 0.1 rpy=0 0 0 -> xyz=0 0 0.1365 rpy=0 0 0

Commit message: Reduced path angle and prefer forward critic weights. increased SLAM transform timeout, minimum travel heading, and loop match minimum; decreased map update interval and added minimum time interval.

File: rover_ws/src/rover_bringup/urdf/rover.urdf (robot description, URDF)
Before this commit: robot rover, 5 links, 4 joints
Joints:
- joint base_to_laser: origin xyz=0 0 0.1365 rpy=0 0 0 -> xyz=0.075 0 0.1365 rpy=0 0 0
- joint base_to_left_wheel: origin xyz=0 0.09 0 rpy=-1.5708 0 0 -> xyz=0 0.09375 0 rpy=-1.5708 0 0
- joint base_to_right_wheel: origin xyz=0 -0.09 0 rpy=-1.5708 0 0 -> xyz=0 -0.09375 0 rpy=-1.5708 0 0
